File: electronics/SSTForkMountBrushedServo/PiHat/RPi_GPIO.sch (KiCad schematic (older format))
At the start: 1 part, among them J2 RPi_GPIO

Commit message: Stepper and Brushed Servo boards, stepper uses toshiba driver.
Parts:
- J2: symbol RPi_GPIO -> RPi_Hat-rescue:RPi_GPIO
Connections:
- wire segments 14 -> 15
Changed lines of the file:
@@
-EESchema Schematic File Version 2
-LIBS:RPi_Hat-rescue
-LIBS:power
-LIBS:device
-LIBS:transistors
-LIBS:conn
-LIBS:linear
-LIBS:regul
-LIBS:74xx
-LIBS:cmos4000
-LIBS:adc-dac
-LIBS:memory
-LIBS:xilinx
-LIBS:microcontrollers
-LIBS:dsp
-LIBS:microchip
-LIBS:analog_switches
-LIBS:motorola
-LIBS:texas
-LIBS:intel
-LIBS:audio
-LIBS:interface
-LIBS:digital-audio
-LIBS:philips
-LIBS:display
-LIBS:cypress
-LIBS:siliconi
-LIBS:opto
-LIBS:atmel
-LIBS:contrib
-LIBS:valves
-LIBS:isadore_custom_components
-LIBS:RPi_Hat-cache
-EELAYER 25 0
+EESchema Schematic File Version 4
+EELAYER 30 0
 EELAYER END
 $Descr A4 11693 8268
@@
 $EndDescr
 $Comp
-L RPi_GPIO J2
+L RPi_Hat-rescue:RPi_GPIO J2
 U 1 1 5516AE26
 P 7500 2700
@@
 	9200 3100 9300 3100
 $Comp
-L +5V #PWR023
+L RPi_Hat-rescue:+5V #PWR023
 U 1 1 5B0302F7
 P 9300 2700
@@
 $EndComp
 Wire Wire Line
-	9200 2700 9300 2700
+	9200 2700 9250 2700
 Wire Wire Line
 	9200 2800 9250 2800
@@
 Connection ~ 9250 2700
 $Comp
-L GND #PWR024
+L RPi_Hat-rescue:GND #PWR024
 U 1 1 5B030319
 P 9300 4300
@@
 $EndComp
 $Comp
-L GND #PWR025
+L RPi_Hat-rescue:GND #PWR025
 U 1 1 5B03032F
 P 9350 2850
@@
 $EndComp
 $Comp
-L GND #PWR026
+L RPi_Hat-rescue:GND #PWR026
 U 1 1 5B030345
 P 9300 3300
@@
 $EndComp
 $Comp
-L GND #PWR027
+L RPi_Hat-rescue:GND #PWR027
 U 1 1 5B03035B
 P 9300 3600
@@
 $EndComp
 $Comp
-L GND #PWR028
+L RPi_Hat-rescue:GND #PWR028
 U 1 1 5B030391
 P 7200 3900
@@
 $EndComp
 $Comp
-L GND #PWR029
+L RPi_Hat-rescue:GND #PWR029
 U 1 1 5B0303A7
 P 7200 4600
@@
 $EndComp
 $Comp
-L GND #PWR030
+L RPi_Hat-rescue:GND #PWR030
 U 1 1 5B0303BD
 P 7200 3100
@@
 NoConn ~ 7300 2800
 NoConn ~ 7300 2700
+Wire Wire Line
+	9250 2700 9300 2700
 $EndSCHEMATC
