File: electronics/SSTForkMountBrushedServo/PiHat/RPi_Hat.sch (KiCad schematic (older format))
At the start: 9 parts, among them CON1 BARREL_JACK, J1 RJ12, J3 M1 Encoder, J4 MPWR, J5 M2 Encoder, U1 pololu_MC33926, U2 pololu_D24V22F5, U3 Teensy_3.1

Commit message: Stepper and Brushed Servo boards, stepper uses toshiba driver.
Parts:
- removed J4: MPWR, SparkFun-Connectors:1X02_LOCK_LONGPADS, symbol Conn_01x02
- removed U1: pololu_MC33926, SparkFun-Connectors:1X18, symbol pololu_MC33926-RESCUE-RPi_Hat
- added SW1: SW_DIP_x01, custom_footprints:PWR_SWITCH_RA1H1C112R, symbol Switch:SW_DIP_x01
- added U1: pololu_MC33926, custom_footprints:pololu_mc33926, symbol SST_kicad_sym:pololu_MC33926
- CON1: symbol BARREL_JACK -> RPi_Hat-rescue:BARREL_JACK
- J1: symbol RJ12 -> RPi_Hat-rescue:RJ12
- J3, J5: symbol Conn_01x04 -> RPi_Hat-rescue:Conn_01x04
- R1: symbol R -> RPi_Hat-rescue:R
- U2: symbol pololu_D24V22F5 -> RPi_Hat-rescue:pololu_D24V22F5
- U3: symbol Teensy_3.1 -> RPi_Hat-rescue:Teensy_3.1
Connections:
- net labels added: SWPWR
- net labels removed: PG
- wire segments 77 -> 81
- no-connect marks 19 -> 25
